Commit message: feat: update desc and launch

File: description/diffbot.urdf.xacro (robot description, xacro)
@@ -2,5 +2,5 @@
 <robot xmlns:xacro="http://www.ros.org/wiki/xacro" name="robot">
     <!-- define args -->
-    <xacro:arg name="sim_mode" default="true" />
+    <xacro:arg name="prefix" default="" />
     <!-- Bot core -->
     <xacro:include filename="$(find epti4abot)/description/diffbot_description.urdf.xacro" />
@@ -8,6 +8,6 @@
     <xacro:include filename="$(find epti4abot)/description/diffbot.materials.xacro" />
     <!-- ROS2 Control -->
-    <xacro:include filename="ros2_control.xacro" />
-    <!-- Lidar sim -->
-    <!-- <xacro:include filename="lidar.xacro" /> -->
+    <xacro:include filename="$(find epti4abot)/description/ros2_control.xacro" />
+    <xacro:diffbot prefix="$(arg prefix)" />
+    <xacro:diffbot_ros2_control name="DiffBot" prefix="$(arg prefix)" />
 </robot>

File: description/diffbot_description.urdf.xacro (robot description, xacro)
@@ -11,6 +11,9 @@
         <xacro:property name="wheel_len" value="0.020" />
         <xacro:property name="wheel_radius" value="0.015" />
-        <xacro:property name="z_offset" value="-${base_height/2}" />
-        <!-- Space btw top of beam and the each joint -->
+        <xacro:property name="caster_wheel_mass" value="0.1" /> <!-- arbitrary value for caster wheel
+        mass -->
+        <xacro:property name="caster_wheel_radius" value="0.015" />
+        <xacro:property name="z_offset" value="-${base_height/2}" /> <!-- Space btw top of beam and
+        the each joint -->
         <!-- Base Link -->
         <link name="${prefix}base_link">
@@ -108,4 +111,61 @@
             <origin xyz="${base_width/2 - caster_wheel_radius} 0 ${z_offset}" rpy="0 0 0" />
         </joint>
+        <!-- caster frontal wheel Link -->
+        <link name="${prefix}caster_frontal_wheel">
+            <collision>
+                <origin xyz="0 0 0" rpy="0 0 0" />
+                <geometry>
+                    <sphere radius="${caster_wheel_radius}" />
+                </geometry>
+            </collision>
+            <visual>
+                <origin xyz="0 0 0" rpy="0 0 0" />
+                <geometry>
+                    <sphere radius="${caster_wheel_radius}" />
+                </geometry>
+                <material name="white" />
+            </visual>
+            <inertial>
+                <origin xyz="0 0 0" rpy="0 0 0" />
+                <mass value="${caster_wheel_mass}" />
+                <inertia
+                    ixx="${caster_wheel_mass * 0.4 * (caster_wheel_radius * caster_wheel_radius)}"
+                    ixy="0.0" ixz="0.0"
+                    iyy="${caster_wheel_mass * 0.4 * (caster_wheel_radius * caster_wheel_radius)}"
+                    iyz="0.0"
+                    izz="${caster_wheel_mass * 0.4 * (caster_wheel_radius * caster_wheel_radius)}" />
+            </inertial>
+        </link>
+        <joint name="${prefix}caster_rear_wheel_joint" type="fixed">
+            <parent link="${prefix}base_link" />
+            <child link="${prefix}caster_rear_wheel" />
+            <origin xyz="${-base_width/2 + caster_wheel_radius} 0 ${z_offset}" rpy="0 0 0" />
+        </joint>
+        <!-- caster rear wheel Link -->
+        <link name="${prefix}caster_rear_wheel">
+            <collision>
+                <origin xyz="0 0 0" rpy="0 0 0" />
+                <geometry>
+                    <sphere radius="${caster_wheel_radius}" />
+                </geometry>
+            </collision>
+            <visual>
+                <origin xyz="0 0 0" rpy="0 0 0" />
+                <geometry>
+                    <sphere radius="${caster_wheel_radius}" />
+                </geometry>
+                <material name="white" />
+            </visual>
+            <inertial>
+                <origin xyz="0 0 0" rpy="0 0 0" />
+                <mass value="${caster_wheel_mass}" />
+                <inertia
+                    ixx="${caster_wheel_mass * 0.4 * (caster_wheel_radius * caster_wheel_radius)}"
+                    ixy="0.0" ixz="0.0"
+                    iyy="${caster_wheel_mass * 0.4 * (caster_wheel_radius * caster_wheel_radius)}"
+                    iyz="0.0"
+                    izz="${caster_wheel_mass * 0.4 * (caster_wheel_radius * caster_wheel_radius)}" />
+            </inertial>
+        </link>
     </xacro:macro>
 </robot>

File: description/ros2_control.xacro (robot description, xacro)
@@ -1,49 +1,22 @@
 <?xml version="1.0"?>
 <robot xmlns:xacro="http://www.ros.org/wiki/xacro">
-    <xacro:unless value="$(arg sim_mode)">
-        <ros2_control name="RealRobot" type="system">
+    <xacro:macro name="diffbot_ros2_control" params="name prefix">
+        <ros2_control name="${name}" type="system">
             <hardware>
-                <!-- TODO -->
+                <plugin>epti4abot/Dfrobot</plugin>
+                <param name="example_param_hw_start_duration_sec">0</param>
+                <param name="example_param_hw_stop_duration_sec">3.0</param>
             </hardware>
-            <joint name="left_wheel_joint">
-                <command_interface name="velocity">
-                    <param name="min">-10</param>
-                    <param name="max">10</param>
-                </command_interface>
+            <joint name="${prefix}left_wheel_joint">
+                <command_interface name="velocity" />
+                <state_interface name="position" />
                 <state_interface name="velocity" />
+            </joint>
+            <joint name="${prefix}right_wheel_joint">
+                <command_interface name="velocity" />
                 <state_interface name="position" />
-            </joint>
-            <joint name="right_wheel_joint">
-                <command_interface name="velocity">
-                    <param name="min">-10</param>
-                    <param name="max">10</param>
-                </command_interface>
                 <state_interface name="velocity" />
-                <state_interface name="position" />
             </joint>
         </ros2_control>
-    </xacro:unless>
-    <xacro:if value="$(arg sim_mode)">
-        <ros2_control name="GazeboSystem" type="system">
-            <hardware>
-                <plugin>gazebo_ros2_control/GazeboSystem</plugin>
-            </hardware>
-            <joint name="left_wheel_joint">
-                <command_interface name="velocity">
-                    <param name="min">-10</param>
-                    <param name="max">10</param>
-                </command_interface>
-                <state_interface name="velocity" />
-                <state_interface name="position" />
-            </joint>
-            <joint name="right_wheel_joint">
-                <command_interface name="velocity">
-                    <param name="min">-10</param>
-                    <param name="max">10</param>
-                </command_interface>
-                <state_interface name="velocity" />
-                <state_interface name="position" />
-            </joint>
-        </ros2_control>
-    </xacro:if>
+    </xacro:macro>
 </robot>
